Commit message: added lidar to the robot and change the mass of the robot

File: urdf/my_robot_integration.urdf.xacro (robot description, xacro)
@@ -5,5 +5,5 @@
 	<!-- Include Robot's urdf filepath -->
 	<!-- Include Lidar's urdf filepath -->
-	<xacro:include filename="$(find proj_1_662)/urdf/car.urdf"/>
+	<xacro:include filename="$(find proj_1_662)/urdf/Assem3.urdf"/>
 	<xacro:include filename="$(find proj_1_662)/urdf/ydlidar.urdf"/>
 <!-- Add your gazebo sensors here -->
@@ -46,14 +46,32 @@
 <!--  Gazebo plugin for control here is already added for you -->
 	<gazebo>
+		<plugin name="differential_drive_controller" filename="libgazebo_ros_diff_drive.so">
+		<alwaysOn>false</alwaysOn>
+		<robotNamespace>/my_robot</robotNamespace>
+		<commandTopic>/my_robot/mobile_base_controller/cmd_vel</commandTopic>
+		<odometryTopic>/my_robot/mobile_base_controller/odom</odometryTopic>
+		<rosDebugLevel>Debug</rosDebugLevel>
+		<publishWheelTF>True</publishWheelTF>
+		<publishWheelJointState>true</publishWheelJointState>
+		<publishTf>1</publishTf>
+		<legacyMode>false</legacyMode>
+		<updateRate>20</updateRate>
+		<leftJoint>left_wheel_joint</leftJoint>
+		<rightJoint>right_wheel_joint</rightJoint>
+		<wheelSeparation>0.1</wheelSeparation>
+		<wheelDiameter>0.5</wheelDiameter>
+		<wheelTorque>5</wheelTorque>
+		<robotBaseFrame>base_link</robotBaseFrame>
+		</plugin>
 		<plugin name="gazebo_ros_control" filename="libgazebo_ros_control.so">
-			<robotNamespace>/simple_car</robotNamespace>
+			<robotNamespace>/my_robot</robotNamespace>
 			<robotSimType>gazebo_ros_control/DefaultRobotHWSim</robotSimType>
 			<legacyModeNS>true</legacyModeNS>
 		</plugin>
-	</gazebo>
+  	</gazebo>
 <!-- Create a joint between your robot and sensor -->
 	<joint name="ylidar" type="fixed">
-		<axis xyz="0 1 0"/>
-		<origin xyz="0.15 0 0.1" rpy="0 0 0" />
+		<!-- <axis xyz="0 1 0"/> -->
+		<origin xyz="0.1 0 0.03" rpy="0 0 0" />
 		<parent link="base_link"/>
 		<child link="base_laser"/>
