Commit message: add README.md and change the mass of the robot model

File: urdf/my_robot_ydlidar.urdf (robot description, URDF)
Before this commit: robot car, 7 links, 6 joints
Links:
- link base_link: mass 9 -> 5
- link castor_wheel: mass 0.5 -> 1
- link laser_frame: mass 0.25482 -> 0.0001
- link left_wheel: mass 0.5 -> 2
- link right_wheel: mass 0.5 -> 2
Joints:
- joint castor_wheel_joint: type continuous -> fixed
